Commit message: Removing collision and increase camera resolution

File: realsense2_description/urdf/_d435.gazebo.xacro (robot description, xacro)
@@ -27,6 +27,6 @@
           <horizontal_fov>${69.4*deg_to_rad}</horizontal_fov>
           <image>
-            <width>640</width>
-            <height>480</height>
+            <width>1280</width>
+            <height>720</height>
             <format>RGB_INT8</format>
           </image>

File: realsense2_description/urdf/_d435.urdf.xacro (robot description, xacro)
@@ -65,10 +65,11 @@
         </xacro:unless>
       </visual>
-      <collision>
+      <!-- Remove collision for integration purposes -->
+      <!--collision>
         <origin xyz="0 ${-d435_cam_depth_py} 0" rpy="0 0 0"/>
         <geometry>
           <box size="${d435_cam_depth} ${d435_cam_width} ${d435_cam_height}"/>
         </geometry>
-      </collision>
+      </collision-->
       <inertial>
         <!-- The following are not reliable values, and should not be used for modeling -->

Commit message: Update camera characteristics to match OAK-D camera

File: realsense2_description/urdf/_d435.gazebo.xacro (robot description, xacro)
@@ -25,5 +25,5 @@
       <sensor name="${camera_name}color" type="camera">
         <camera name="${camera_name}">
-          <horizontal_fov>${69.4*deg_to_rad}</horizontal_fov>
+          <horizontal_fov>${50.41*deg_to_rad}</horizontal_fov>
           <image>
             <width>1280</width>
@@ -47,8 +47,8 @@
       <sensor name="${camera_name}ired1" type="camera">
         <camera name="${camera_name}">
-          <horizontal_fov>${85.2*deg_to_rad}</horizontal_fov>
+          <horizontal_fov>${52.46*deg_to_rad}</horizontal_fov>
           <image>
             <width>1280</width>
-            <height>720</height>
+            <height>800</height>
             <format>L_INT8</format>
           </image>
@@ -69,8 +69,8 @@
       <sensor name="${camera_name}ired2" type="camera">
         <camera name="${camera_name}">
-          <horizontal_fov>${85.2*deg_to_rad}</horizontal_fov>
+          <horizontal_fov>${52.46*deg_to_rad}</horizontal_fov>
           <image>
             <width>1280</width>
-            <height>720</height>
+            <height>800</height>
             <format>L_INT8</format>
           </image>
@@ -91,8 +91,8 @@
       <sensor name="${camera_name}depth" type="depth">
         <camera name="${camera_name}">
-          <horizontal_fov>${85.2*deg_to_rad}</horizontal_fov>
+          <horizontal_fov>${52.46*deg_to_rad}</horizontal_fov>
           <image>
             <width>1280</width>
-            <height>720</height>
+            <height>800</height>
           </image>
           <clip>
@@ -129,10 +129,10 @@
         <infrared1OpticalframeName>${infrared1_optical_frame}</infrared1OpticalframeName>
         <infrared2OpticalframeName>${infrared2_optical_frame}</infrared2OpticalframeName>
-        <rangeMinDepth>0.2</rangeMinDepth>
-        <rangeMaxDepth>10.0</rangeMaxDepth>
+        <rangeMinDepth>0.35</rangeMinDepth>
+        <rangeMaxDepth>5.5</rangeMaxDepth>
         <pointCloud>${publish_pointcloud}</pointCloud>
         <pointCloudTopicName>depth/color/points</pointCloudTopicName>
-        <pointCloudCutoff>0.25</pointCloudCutoff>
-        <pointCloudCutoffMax>9.0</pointCloudCutoffMax>
+        <pointCloudCutoff>0.4</pointCloudCutoff>
+        <pointCloudCutoffMax>6.0</pointCloudCutoffMax>
       </plugin>
     </gazebo>

File: realsense2_description/urdf/_d435.urdf.xacro (robot description, xacro)
@@ -15,7 +15,7 @@
     <!-- The following values are approximate, and the camera node
      publishing TF values with actual calibrated camera extrinsic values -->
-    <xacro:property name="d435_cam_depth_to_infra1_offset" value="0.0"/>
-    <xacro:property name="d435_cam_depth_to_infra2_offset" value="-0.050"/>
-    <xacro:property name="d435_cam_depth_to_color_offset" value="0.015"/>
+    <xacro:property name="d435_cam_depth_to_infra1_offset" value="0.075"/>
+    <xacro:property name="d435_cam_depth_to_infra2_offset" value="-0.075"/>
+    <xacro:property name="d435_cam_depth_to_color_offset" value="0.0"/>
     <!-- The following values model the aluminum peripherial case for the
   	D435 camera, with the camera joint represented by the actual

Commit message: Add true stereo to D435 in realsense2_description
All the cameras were originally set on camera_link, but each of the infrared cameras should be on their respective frames to get stereo feeds

File: realsense2_description/urdf/_d435.gazebo.xacro (robot description, xacro)
@@ -6,5 +6,9 @@
 -->
 <robot xmlns:xacro="http://ros.org/wiki/xacro">
-  <xacro:macro name="gazebo_d435" params="camera_name reference_link topics_ns depth_optical_frame color_optical_frame infrared1_optical_frame infrared2_optical_frame publish_pointcloud:=true" >
+  <xacro:macro name="gazebo_d435"
+    params="camera_name reference_link topics_ns
+    depth_optical_frame color_optical_frame infrared1_optical_frame infrared2_optical_frame
+    depth_frame color_frame infrared1_frame infrared2_frame
+    publish_pointcloud:=true" >
     <!-- Load parameters to model's main link-->
     <xacro:property name="deg_to_rad" value="0.01745329251994329577" />
@@ -13,5 +17,5 @@
       <enable_wind>0</enable_wind>
       <kinematic>0</kinematic>
-      <gravity>1</gravity>
+      <!-- <gravity>1</gravity> -->
       <!--<mu>1</mu>-->
       <mu2>1</mu2>
@@ -23,4 +27,6 @@
       <!--<max_vel>0.01</max_vel>
       <min_depth>0</min_depth>-->
+    </gazebo>
+    <gazebo reference="${color_frame}">
       <sensor name="${camera_name}color" type="camera">
         <camera name="${camera_name}">
@@ -45,4 +51,6 @@
         <visualize>1</visualize>
       </sensor>
+    </gazebo>
+    <gazebo reference="${infrared1_frame}">
       <sensor name="${camera_name}ired1" type="camera">
         <camera name="${camera_name}">
@@ -67,4 +75,6 @@
         <visualize>0</visualize>
       </sensor>
+    </gazebo>
+    <gazebo reference="${infrared2_frame}">
       <sensor name="${camera_name}ired2" type="camera">
         <camera name="${camera_name}">
@@ -89,4 +99,6 @@
         <visualize>0</visualize>
       </sensor>
+    </gazebo>
+    <gazebo reference="${depth_frame}">
       <sensor name="${camera_name}depth" type="depth">
         <camera name="${camera_name}">

File: realsense2_description/urdf/_d435.urdf.xacro (robot description, xacro)
@@ -140,5 +140,10 @@
     </xacro:if>
     <!-- Realsense Gazebo Plugin -->
-    <xacro:gazebo_d435 camera_name="${name}" reference_link="${name}_link" topics_ns="${topics_ns}" depth_optical_frame="${name}_depth_optical_frame" color_optical_frame="${name}_color_optical_frame" infrared1_optical_frame="${name}_left_ir_optical_frame" infrared2_optical_frame="${name}_right_ir_optical_frame" publish_pointcloud="${publish_pointcloud}"/>
+    <xacro:gazebo_d435 camera_name="${name}" reference_link="${name}_link" topics_ns="${topics_ns}"
+      depth_optical_frame="${name}_depth_optical_frame" color_optical_frame="${name}_color_optical_frame"
+      infrared1_optical_frame="${name}_infra1_optical_frame" infrared2_optical_frame="${name}_infra2_optical_frame"
+      depth_frame="${name}_depth_frame" color_frame="${name}_color_frame"
+      infrared1_frame="${name}_infra1_frame" infrared2_frame="${name}_infra2_frame"
+      publish_pointcloud="${publish_pointcloud}" />
   </xacro:macro>
 </robot>
